File: 3340.kicad_sch (KiCad schematic)
At the start: 181 parts, among them J1 Conn_01x16, J10 FM1, J11 Conn_01x16, J12 V/OCT2, J13 PULSE2, J14 SAW2, J15 TRI2, J16 SINE2, J17 SYNC2, J18 Conn_01x16, J19 PWM2, J2 Conn_01x16, J20 FM2, J3 V/OCT1, J4 PULSE1, J5 SAW1, J6 TRI1, J7 SINE1, J8 SYNC1, J9 PWM1, Q1 2N3904, Q2 2N3906, Q3 2N3904, Q4 2N3906, Q5 2N3904, Q6 2N3904, SW2 DPDT_OOO, U1 TL072, U2 TL074, U3 CEM3340, U4 TL072, U5 CEM3340, U6 TL074

Commit message: Fix power routing
Parts:
- removed C37, C38: 10u, Capacitor_THT:C_Disc_D4.3mm_W1.9mm_P5.00mm, symbol Device:C_Polarized
- removed D7, D8: 1N5818, Diode_THT:D_DO-41_SOD81_P10.16mm_Horizontal, symbol Diode:1N5818
- removed J1, J11, J18, J2: Conn_01x16, Connector_PinHeader_2.54mm:PinHeader_1x16_P2.54mm_Vertical, symbol Connector_Generic:Conn_01x16
- removed PWR2: PWR, Connector_IDC:IDC-Header_2x05_P2.54mm_Vertical, symbol Connector_Generic:Conn_02x05_Odd_Even
- added J? (x4): Conn_01x17, symbol Connector_Generic:Conn_01x17
Connections:
- net +12V: now also J?.3 (Pin_3), J?.3 (Pin_3)
- net -12V: now also J?.1 (Pin_1), J?.1 (Pin_1)
- net 12v: now also J?.3 (Pin_3), J?.3 (Pin_3)
- net COARSE1: now also J?.4 (Pin_4)
- net COARSE2: now also J?.4 (Pin_4)
- net FINE1: now also J?.5 (Pin_5)
- net FINE2: now also J?.5 (Pin_5)
- net FMOD1: now also J?.8 (Pin_8)
- net FMOD2: now also J?.8 (Pin_8)
- net GND: now also J?.2 (Pin_2), J?.2 (Pin_2), J?.2 (Pin_2), J?.2 (Pin_2)
- net PULSEOUT1: now also J?.13 (Pin_13)
- net PULSEOUT2: now also J?.13 (Pin_13)
- net PWM_IN1: now also J?.7 (Pin_7)
- net PWM_IN2: now also J?.7 (Pin_7)
- net PW_IN1: now also J?.6 (Pin_6)
- net PW_IN2: now also J?.6 (Pin_6)
- net SAW1: now also J?.17 (Pin_17)
- net SAW12: now also J?.17 (Pin_17)
- net SAW2: now also J?.17 (Pin_17)
- net SAW21: now also J?.17 (Pin_17)
- net SAWIN1: now also J?.12 (Pin_12)
- net SAWIN2: now also J?.12 (Pin_12)
- net SAWOUT1: now also J?.14 (Pin_14)
- net SAWOUT2: now also J?.14 (Pin_14)
- net SAW_IN1: now also J?.12 (Pin_12)
- net SAW_IN2: now also J?.12 (Pin_12)
- net SHAPE1: now also J?.15 (Pin_15)
- net SHAPE2: now also J?.15 (Pin_15)
- net SINE1: now also J?.16 (Pin_16)
- net SINE2: now also J?.16 (Pin_16)
- net SYNC+1: now also J?.9 (Pin_9)
- net SYNC+2: now also J?.9 (Pin_9)
- net SYNC-1: now also J?.10 (Pin_10)
- net SYNC-2: now also J?.10 (Pin_10)
- net VOCT1: now also J?.11 (Pin_11)
- net VOCT2: now also J?.11 (Pin_11)
- net V/OCT1: now also J?.11 (Pin_11)
- net V/OCT2: now also J?.11 (Pin_11)
- net at J20.T: now also J?.8 (Pin_8)
- net at SNC2.1: now also J?.9 (Pin_9)
- net at SNC2.6: now also J?.10 (Pin_10)
- net at R38.1: now also J?.15 (Pin_15)
- net at J10.T: now also J?.8 (Pin_8)
- net at R73.1: now also J?.13 (Pin_13)
- net at R37.1: now also J?.14 (Pin_14)
- net at PW1.2: now also J?.6 (Pin_6)
- net at PWM2.2: now also J?.7 (Pin_7)
- net at SNC1.1: now also J?.9 (Pin_9)
- net at SNC1.6: now also J?.10 (Pin_10)
- net at PWM1.2: now also J?.7 (Pin_7)
- net at R74.1: now also J?.14 (Pin_14)
- net at R75.1: now also J?.15 (Pin_15)
- net at R36.1: now also J?.13 (Pin_13)
- net at R39.1: now also J?.16 (Pin_16)
- net at COARSE1.2: now also J?.4 (Pin_4)
- net at FINE1.2: now also J?.5 (Pin_5)
- net at PW2.2: now also J?.6 (Pin_6)
- net at COARSE2.2: now also J?.4 (Pin_4)
- net at R76.1: now also J?.16 (Pin_16)
- net at FINE2.2: now also J?.5 (Pin_5)
- new net -12: J?.1 (Pin_1), J?.1 (Pin_1)
